File: EAGLE/LJ-STAND/Main.brd (EAGLE design)
At the start: 160 x 100 mm, 120 parts, among them Q1 BSS138, Q2 BSS138

Commit message: TSOPS placed on pcb and lots of other stuff
Parts:
- removed LED5: GREEN, adafruit:CHIPLED_0603
- added PWR: BLUE, adafruit:CHIPLED_0603
- LED1: value BLUE -> GREEN
- MTR1_OUT, MTR2_OUT, MTR3_OUT: value VH -> PH; device jst-vh:B2P-VH -> adafruit:JST-PH-2-SMT
- moved C42 265.8 mm to (148.6, 196.4)
- moved C10 258.6 mm to (125.5, 239.3)
- moved C43 256.6 mm to (138.5, 181.3)
- moved MOTOR_2 255.0 mm to (81.3, 179.1)
- moved C41 254.8 mm to (132.4, 225.2)
- moved LIGHT_SENSOR_CONNECTOR 246.6 mm to (102.9, 207.6), flipped to the bottom, turned to 90 degrees
- moved 6 244.9 mm to (151.9, 199.1), flipped to the bottom, turned to 270 degrees
- moved SLAVE_TSOP 244.4 mm to (116.8, 199.4)
- moved 7 240.4 mm to (142.3, 182.8), flipped to the bottom, turned to 285 degrees
- moved C13 239.8 mm to (99.1, 234.9), flipped to the bottom, turned to 270 degrees
- moved BLUETOOTH 235.2 mm to (130.8, 191.8), turned to 90 degrees
- moved C40 234.0 mm to (113.0, 227.3), flipped to the bottom
- moved 5 232.7 mm to (142.3, 215.2), flipped to the bottom, turned to 255 degrees
- moved VREG-3.3V 232.6 mm to (108.0, 240.0), flipped to the bottom, turned to 90 degrees
- moved MOTOR_1 232.6 mm to (62.2, 179.1)
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Connections:
- net GND: now also PWR.C; no longer LED5.C
- net N$1: now also MTR2_OUT.1; no longer MTR2_OUT.2
- net N$14: now also MTR3_OUT.1; no longer MTR3_OUT.2
- net N$16: now also MTR3_OUT.2; no longer MTR3_OUT.1
- net N$2: now also MTR2_OUT.2; no longer MTR2_OUT.1
- net N$23: now also LED2.A; no longer LED3.A
- net N$24: now also LED3.A; no longer LED4.A
- net N$25: now also LED4.A; no longer LED5.A
- net N$27: now also PWR.A; no longer LED1.A
- net N$29: now also LED1.A; no longer LED2.A
- net N$5: now also MTR1_OUT.1; no longer MTR1_OUT.2
- net N$7: now also MTR1_OUT.2; no longer MTR1_OUT.1
Other:
- board size 160 x 100 mm -> 158.5 x 133.6 mm

Commit message: PCB Routing
Parts:
- removed Q1, Q2: BSS138, m-pad-2.1:SOT23
- removed XBEE: XBEE, adafruit:XBEE
- added SCL, SDA: BSS138, m-pad-2.1:SOT23
- moved C5 119.9 mm to (112.8, 260.1), turned to 180 degrees
- moved C6 119.5 mm to (126.4, 248.0), flipped to the top, turned to 180 degrees
- moved C9 114.9 mm to (155.8, 202.3), turned to 90 degrees
- moved C39 105.1 mm to (42.7, 227.3)
- moved C24 95.6 mm to (62.2, 171.4), flipped to the bottom, turned to 90 degrees
- moved C8 95.0 mm to (145.0, 218.0), flipped to the top, turned to 90 degrees
- moved C7 93.0 mm to (136.0, 232.8), flipped to the top, turned to 90 degrees
- moved C3 89.4 mm to (78.3, 257.8), flipped to the top, turned to 180 degrees
- moved C4 88.5 mm to (94.7, 258.9), flipped to the top, turned to 180 degrees
- moved C38 88.4 mm to (113.4, 227.6), flipped to the bottom
- moved C41 71.6 mm to (130.3, 153.7)
- moved C29 70.9 mm to (81.3, 171.4), flipped to the bottom, turned to 90 degrees
- moved R17 65.9 mm to (62.2, 236.2), turned to 270 degrees
- moved C42 65.7 mm to (121.0, 136.7)
- moved R20 64.3 mm to (31.8, 181.6), turned to 0 degrees
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Connections:
- net +3V3: now also SCL.1, SDA.1; no longer Q1.1, Q2.1, XBEE.1
- net GND: no longer XBEE.10
- net SCL: now also SCL.2; no longer Q1.2
- net SCL_5V: now also SCL.3; no longer Q1.3
- net SDA: now also SDA.2; no longer Q2.2
- net SDA_5V: now also SDA.3; no longer Q2.3
- net XBEE_RX: no longer XBEE.3
- net XBEE_TX: no longer XBEE.2
Routing:
- net TSOP_PWR: track 0.00 -> 546.5 mm
- net TSOP14: track 0.00 -> 142.8 mm, vias 0 -> 1
- net TSOP15: track 0.00 -> 126.5 mm, vias 0 -> 1
- net TSOP13: track 0.00 -> 121.6 mm
- net +5V: track 0.00 -> 108.9 mm
- net TSOP12: track 0.00 -> 103.8 mm
- net TSOP10: track 0.00 -> 97.7 mm
- net GND: track 0.00 -> 96.0 mm, vias 0 -> 1
- net TSOP11: track 0.00 -> 86.7 mm
- net TSOP9: track 0.00 -> 81.6 mm
- net TSOP8: track 0.00 -> 69.0 mm
- net TSOP7: track 0.00 -> 62.8 mm
- net TSOP0: track 0.00 -> 62.3 mm
- net TSOP6: track 0.00 -> 55.6 mm
- net TSOP1: track 0.00 -> 51.2 mm
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- added copper zone on layer 16, net GND
Other:
- outline, holes or cut-outs redrawn
