File: EAGLE/LJ-STAND/Main.sch (EAGLE design)
At the start: 78 parts

Commit message: Things
Parts:
- renumbered MTR2_OUT1 to MTR2_OUT, MTR3_OUT2 to MTR3_OUT
Changed lines of the file:
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@@
 <part name="GND51" library="supply1" deviceset="GND" device=""/>
 <part name="C29" library="SparkFun-Capacitors" deviceset="CAP" device="0603-CAP" value="0.1uF"/>
-<part name="MTR2_OUT1" library="jst-vh" deviceset="B2P-VH" device=""/>
+<part name="MTR2_OUT" library="jst-vh" deviceset="B2P-VH" device=""/>
 <part name="C30" library="SparkFun-Capacitors" deviceset="CAP" device="0603-CAP" value="0.01uF"/>
 <part name="C31" library="SparkFun-Capacitors" deviceset="CAP" device="0603-CAP" value="0.22uF"/>
@@
 <part name="GND56" library="supply1" deviceset="GND" device=""/>
 <part name="C34" library="SparkFun-Capacitors" deviceset="CAP" device="0603-CAP" value="0.1uF"/>
-<part name="MTR3_OUT2" library="jst-vh" deviceset="B2P-VH" device=""/>
+<part name="MTR3_OUT" library="jst-vh" deviceset="B2P-VH" device=""/>
 <part name="C35" library="SparkFun-Capacitors" deviceset="CAP" device="0603-CAP" value="0.01uF"/>
 <part name="C36" library="SparkFun-Capacitors" deviceset="CAP" device="0603-CAP" value="0.22uF"/>
@@
 <instance part="GND51" gate="1" x="256.54" y="208.28"/>
 <instance part="C29" gate="G$1" x="243.84" y="200.66" rot="R90"/>
-<instance part="MTR2_OUT1" gate="G$1" x="243.84" y="190.5" rot="R270"/>
+<instance part="MTR2_OUT" gate="G$1" x="243.84" y="190.5" rot="R270"/>
 <instance part="C30" gate="G$1" x="220.98" y="241.3" rot="R180"/>
 <instance part="C31" gate="G$1" x="220.98" y="254" rot="R180"/>
@@
 <instance part="GND56" gate="1" x="172.72" y="210.82"/>
 <instance part="C34" gate="G$1" x="160.02" y="203.2" rot="R90"/>
-<instance part="MTR3_OUT2" gate="G$1" x="160.02" y="193.04" rot="R270"/>
+<instance part="MTR3_OUT" gate="G$1" x="160.02" y="193.04" rot="R270"/>
 <instance part="C35" gate="G$1" x="137.16" y="243.84" rot="R180"/>
 <instance part="C36" gate="G$1" x="137.16" y="256.54" rot="R180"/>
@@
 <wire x1="226.06" y1="200.66" x2="236.22" y2="200.66" width="0.1524" layer="91"/>
 <pinref part="C29" gate="G$1" pin="1"/>
-<pinref part="MTR2_OUT1" gate="G$1" pin="2"/>
+<pinref part="MTR2_OUT" gate="G$1" pin="2"/>
 <wire x1="236.22" y1="200.66" x2="238.76" y2="200.66" width="0.1524" layer="91"/>
 <wire x1="241.3" y1="190.5" x2="241.3" y2="195.58" width="0.1524" layer="91"/>
@@
 <wire x1="261.62" y1="200.66" x2="248.92" y2="200.66" width="0.1524" layer="91"/>
 <pinref part="C29" gate="G$1" pin="2"/>
-<pinref part="MTR2_OUT1" gate="G$1" pin="1"/>
+<pinref part="MTR2_OUT" gate="G$1" pin="1"/>
 <wire x1="248.92" y1="200.66" x2="246.38" y2="200.66" width="0.1524" layer="91"/>
 <wire x1="243.84" y1="190.5" x2="243.84" y2="195.58" width="0.1524" layer="91"/>
@@
 <wire x1="142.24" y1="203.2" x2="152.4" y2="203.2" width="0.1524" layer="91"/>
 <pinref part="C34" gate="G$1" pin="1"/>
-<pinref part="MTR3_OUT2" gate="G$1" pin="2"/>
+<pinref part="MTR3_OUT" gate="G$1" pin="2"/>
 <wire x1="152.4" y1="203.2" x2="154.94" y2="203.2" width="0.1524" layer="91"/>
 <wire x1="157.48" y1="193.04" x2="157.48" y2="198.12" width="0.1524" layer="91"/>
@@
 <wire x1="177.8" y1="203.2" x2="165.1" y2="203.2" width="0.1524" layer="91"/>
 <pinref part="C34" gate="G$1" pin="2"/>
-<pinref part="MTR3_OUT2" gate="G$1" pin="1"/>
+<pinref part="MTR3_OUT" gate="G$1" pin="1"/>
 <wire x1="165.1" y1="203.2" x2="162.56" y2="203.2" width="0.1524" layer="91"/>
 <wire x1="160.02" y1="193.04" x2="160.02" y2="198.12" width="0.1524" layer="91"/>

Commit message: Stuffs
Parts:
- added Q1, Q2: BSS138, m-pad-2.1:BSS138
- VREG-3.3V: value LM340S-05 -> LM1084
Connections:
- new net TEENSY_SDL: TSOP.37/A18/PWM/SCL1
- net N$21: no longer MOTOR_FUSE.P2A
- net N$9: no longer LOGIC_FUSE.P2A
- net PWR: no longer LOGIC_FUSE.P1A, MOTOR_FUSE.P1A
- net TEENSY_SCL: now also LIGHT_SENSOR.3/PWM/CAN0TX/SCL2
- net TEENSY_SDA: now also LIGHT_SENSOR.4/PWM/CAN0RX/SDA2, TSOP.38/A19/PWM/SDA1
Changed lines of the file:
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@@
 <?xml version="1.0" encoding="utf-8"?>
 <!DOCTYPE eagle SYSTEM "eagle.dtd">
-<eagle version="7.5.0">
+<eagle version="7.2.0">
 <drawing>
 <settings>
@@
 </classes>
 <parts>
-<part name="MOTOR_FUSE" library="fuse-holder-3568" deviceset="3568-FUSEHOLDER" device="" value="7.5A"/>
-<part name="LOGIC_FUSE" library="fuse-holder-3568" deviceset="3568-FUSEHOLDER" device="" value="2A"/>
 <part name="C1" library="SparkFun-Capacitors" deviceset="CAP_POL" device="PTH4" value="1000uF"/>
 <part name="GND1" library="supply1" deviceset="GND" device=""/>
@@
 <part name="C12" library="SparkFun-Capacitors" deviceset="CAP" device="0805" value="22uF"/>
 <part name="P+1" library="supply1" deviceset="+5V" device=""/>
-<part name="VREG-3.3V" library="linear" deviceset="LM340?-*" device="S" technology="05"/>
+<part name="VREG-3.3V" library="linear" deviceset="LM340?-*" device="S" technology="05" value="LM1084"/>
 <part name="GND9" library="supply1" deviceset="GND" device=""/>
 <part name="+3V1" library="supply1" deviceset="+3V3" device=""/>
@@
 <part name="P+3" library="supply1" deviceset="+5V" device=""/>
 <part name="GND74" library="supply1" deviceset="GND" device=""/>
+<part name="MOTOR_FUSE" library="fuse-holder-3568" deviceset="3568-FUSEHOLDER" device="" value="7.5A"/>
+<part name="LOGIC_FUSE" library="fuse-holder-3568" deviceset="3568-FUSEHOLDER" device="" value="2A"/>
+<part name="Q1" library="m-pad-2.1" deviceset="BSS138" device=""/>
+<part name="Q2" library="m-pad-2.1" deviceset="BSS138" device=""/>
 </parts>
 <sheets>
@@
 </plain>
 <instances>
-<instance part="MOTOR_FUSE" gate="G$1" x="50.8" y="73.66"/>
-<instance part="LOGIC_FUSE" gate="G$1" x="50.8" y="55.88"/>
 <instance part="C1" gate="G$1" x="25.4" y="63.5"/>
 <instance part="GND1" gate="1" x="27.94" y="53.34"/>
@@
 <instance part="C13" gate="G$1" x="124.46" y="48.26"/>
 <instance part="C14" gate="G$1" x="154.94" y="48.26"/>
-<instance part="MOTOR_SWITCH" gate="G$1" x="71.12" y="78.74" rot="R90"/>
-<instance part="LOGIC_SWITCH" gate="G$1" x="71.12" y="50.8" rot="R270"/>
+<instance part="MOTOR_SWITCH" gate="G$1" x="71.12" y="78.74" smashed="yes" rot="R90">
+<attribute name="NAME" x="90.17" y="85.09" size="1.778" layer="95" rot="R180"/>
+<attribute name="VALUE" x="78.74" y="74.93" size="1.778" layer="96" rot="R90"/>
+</instance>
+<instance part="LOGIC_SWITCH" gate="G$1" x="71.12" y="50.8" smashed="yes" rot="R270">
+<attribute name="NAME" x="54.61" y="44.45" size="1.778" layer="95"/>
+<attribute name="VALUE" x="63.5" y="54.61" size="1.778" layer="96" rot="R270"/>
+</instance>
 <instance part="MASTER" gate="G$1" x="43.18" y="-101.6"/>
 <instance part="GND10" gate="1" x="5.08" y="-5.08"/>
@@
 <instance part="P+3" gate="1" x="78.74" y="149.86"/>
 <instance part="GND74" gate="1" x="73.66" y="129.54"/>
+<instance part="MOTOR_FUSE" gate="G$1" x="50.8" y="71.12"/>
+<instance part="LOGIC_FUSE" gate="G$1" x="50.8" y="53.34"/>
+<instance part="Q1" gate="G$1" x="332.74" y="106.68" rot="R90"/>
+<instance part="Q2" gate="G$1" x="309.88" y="106.68" rot="R90"/>
 </instances>
 <busses>
@@
 <segment>
 <pinref part="C1" gate="G$1" pin="+"/>
-<pinref part="MOTOR_FUSE" gate="G$1" pin="P1"/>
-<wire x1="40.64" y1="76.2" x2="38.1" y2="76.2" width="0.1524" layer="91"/>
 <wire x1="25.4" y1="66.04" x2="38.1" y2="66.04" width="0.1524" layer="91"/>
 <wire x1="38.1" y1="66.04" x2="38.1" y2="73.66" width="0.1524" layer="91"/>
 <junction x="25.4" y="66.04"/>
-<pinref part="MOTOR_FUSE" gate="G$1" pin="P1A"/>
-<wire x1="38.1" y1="73.66" x2="38.1" y2="76.2" width="0.1524" layer="91"/>
 <wire x1="40.64" y1="73.66" x2="38.1" y2="73.66" width="0.1524" layer="91"/>
-<junction x="38.1" y="73.66"/>
-<wire x1="38.1" y1="66.04" x2="38.1" y2="58.42" width="0.1524" layer="91"/>
+<wire x1="38.1" y1="66.04" x2="38.1" y2="55.88" width="0.1524" layer="91"/>
 <junction x="38.1" y="66.04"/>
-<pinref part="LOGIC_FUSE" gate="G$1" pin="P1"/>
-<wire x1="38.1" y1="58.42" x2="40.64" y2="58.42" width="0.1524" layer="91"/>
-<wire x1="38.1" y1="58.42" x2="38.1" y2="55.88" width="0.1524" layer="91"/>
-<junction x="38.1" y="58.42"/>
-<pinref part="LOGIC_FUSE" gate="G$1" pin="P1A"/>
 <wire x1="38.1" y1="55.88" x2="40.64" y2="55.88" width="0.1524" layer="91"/>
 <pinref part="PWR_IN" gate="G$1" pin="2"/>
 <wire x1="15.24" y1="66.04" x2="25.4" y2="66.04" width="0.1524" layer="91"/>
+<pinref part="MOTOR_FUSE" gate="G$1" pin="P1"/>
+<pinref part="LOGIC_FUSE" gate="G$1" pin="P1"/>
 </segment>
 </net>
@@
 <net name="N$9" class="0">
 <segment>
-<pinref part="LOGIC_FUSE" gate="G$1" pin="P2"/>
-<wire x1="60.96" y1="58.42" x2="63.5" y2="58.42" width="0.1524" layer="91"/>
-<wire x1="63.5" y1="58.42" x2="63.5" y2="55.88" width="0.1524" layer="91"/>
-<pinref part="LOGIC_FUSE" gate="G$1" pin="P2A"/>
-<wire x1="60.96" y1="55.88" x2="63.5" y2="55.88" width="0.1524" layer="91"/>
-<wire x1="63.5" y1="55.88" x2="68.58" y2="55.88" width="0.1524" layer="91"/>
-<junction x="63.5" y="55.88"/>
+<wire x1="60.96" y1="55.88" x2="68.58" y2="55.88" width="0.1524" layer="91"/>
 <pinref part="LOGIC_SWITCH" gate="G$1" pin="2"/>
 <wire x1="68.58" y1="55.88" x2="68.58" y2="50.8" width="0.1524" layer="91"/>
+<pinref part="LOGIC_FUSE" gate="G$1" pin="P2"/>
 </segment>
 </net>
@@
 <net name="N$21" class="0">
 <segment>
+<pinref part="MOTOR_SWITCH" gate="G$1" pin="1"/>
+<wire x1="60.96" y1="73.66" x2="71.12" y2="73.66" width="0.1524" layer="91"/>
+<wire x1="71.12" y1="73.66" x2="71.12" y2="78.74" width="0.1524" layer="91"/>
 <pinref part="MOTOR_FUSE" gate="G$1" pin="P2"/>
-<wire x1="60.96" y1="76.2" x2="63.5" y2="76.2" width="0.1524" layer="91"/>
-<wire x1="63.5" y1="76.2" x2="63.5" y2="73.66" width="0.1524" layer="91"/>
-<pinref part="MOTOR_SWITCH" gate="G$1" pin="1"/>
-<wire x1="63.5" y1="73.66" x2="71.12" y2="73.66" width="0.1524" layer="91"/>
-<wire x1="71.12" y1="73.66" x2="71.12" y2="78.74" width="0.1524" layer="91"/>
-<pinref part="MOTOR_FUSE" gate="G$1" pin="P2A"/>
-<wire x1="60.96" y1="73.66" x2="63.5" y2="73.66" width="0.1524" layer="91"/>
-<junction x="63.5" y="73.66"/>
 </segment>
 </net>
@@
 <label x="330.2" y="55.88" size="1.778" layer="95" rot="R270" xref="yes"/>
 </segment>
+<segment>
+<pinref part="TSOP" gate="G$1" pin="38/A19/PWM/SDA1"/>
+<wire x1="203.2" y1="-96.52" x2="205.74" y2="-96.52" width="0.1524" layer="91"/>
+<label x="205.74" y="-96.52" size="1.778" layer="95" xref="yes"/>
+</segment>
+<segment>
+<pinref part="LIGHT_SENSOR" gate="G$1" pin="4/PWM/CAN0RX/SDA2"/>
+<wire x1="276.86" y1="-30.48" x2="274.32" y2="-30.48" width="0.1524" layer="91"/>
+<label x="274.32" y="-30.48" size="1.778" layer="95" rot="R180" xref="yes"/>
+</segment>
 </net>
 <net name="TEENSY_SCL" class="0">
@@
 <label x="317.5" y="55.88" size="1.778" layer="95" rot="R270" xref="yes"/>
 </segment>
+<segment>
+<pinref part="LIGHT_SENSOR" gate="G$1" pin="3/PWM/CAN0TX/SCL2"/>
+<wire x1="276.86" y1="-25.4" x2="274.32" y2="-25.4" width="0.1524" layer="91"/>
+<label x="274.32" y="-25.4" size="1.778" layer="95" rot="R180" xref="yes"/>
+</segment>
 </net>
 <net name="PIXY_MISO" class="0">
@@
 </segment>
 </net>
+<net name="TEENSY_SDL" class="0">
+<segment>
+<pinref part="TSOP" gate="G$1" pin="37/A18/PWM/SCL1"/>
+<wire x1="203.2" y1="-101.6" x2="205.74" y2="-101.6" width="0.1524" layer="91"/>
+<label x="205.74" y="-101.6" size="1.778" layer="95" xref="yes"/>
+</segment>
+</net>

Commit message: Logic level converters
Parts:
- added C40, C41, C42, C43, C44, C45, C46, C47: 0.1uF, SparkFun-Capacitors:CAP0603-CAP
- added R5, R6, R7, R8: 10K, SparkFun-Resistors:RESISTOR0603-RES
- added TSOP17, TSOP18, TSOP19, TSOP20, TSOP21, TSOP22, TSOP23, TSOP24: TSOP1737, tsop:TSOP1737
Connections:
- removed net LS25: LIGHT_SENSOR.50/A24
- removed net PIXY_SCL: PIXY_I2C.5
- removed net PIXY_SDA: PIXY_I2C.9
- new net SENSOR_SCL_5V: PIXY_I2C.5, Q1.D, R8.1
- new net SENSOR_SDA_5V: PIXY_I2C.9, Q2.D, R6.1
- new net TSOP17: TSOP.20/A6/PWM/CS0, TSOP17.OUT
- new net TSOP18: TSOP.21/A7/PWM/CS0, TSOP18.OUT
- new net TSOP19: TSOP.22/A8/PWM, TSOP19.OUT
- new net TSOP20: TSOP.23/A9/PWM, TSOP20.OUT
- new net TSOP21: TSOP.24, TSOP21.OUT
- new net TSOP22: TSOP.25, TSOP22.OUT
- new net TSOP23: TSOP.26, TSOP23.OUT
- new net TSOP24: TSOP.27, TSOP24.OUT
- net +3V3: now also Q1.G, Q2.G, R5.2, R7.2
- net +5V: now also R6.2, R8.2
- net GND: now also C40.2, C41.2, C42.2, C43.2, C44.2, C45.2, C46.2, C47.2, TSOP17.GND, TSOP18.GND, TSOP19.GND, TSOP20.GND, TSOP21.GND, TSOP22.GND, TSOP23.GND, TSOP24.GND
- net SENSOR_SCL: now also Q1.S, R7.1
- net SENSOR_SDA: now also Q2.S, R5.1
- net TSOP_PWR: now also C40.1, C41.1, C42.1, C43.1, C44.1, C45.1, C46.1, C47.1, TSOP.28, TSOP.29/PWM, TSOP.30/PWM, TSOP.31/A12/RX4/CS1, TSOP17.V+, TSOP18.V+, TSOP19.V+, TSOP20.V+, TSOP21.V+, TSOP22.V+, TSOP23.V+, TSOP24.V+; no longer TSOP.20/A6/PWM/CS0, TSOP.21/A7/PWM/CS0, TSOP.22/A8/PWM, TSOP.23/A9/PWM
Other:
- moved on the sheet: C38, Q1, Q2

Commit message: PCB
Parts:
- removed LIGHT_SENSOR, TSOP: TEENSY-3.5, teensy-3.5:TEENSY-3.5
- added BLUETOOTH: (no value), SparkFun-Connectors:M06SILK_FEMALE_PTH
- added LED1: BLUE, adafruit:LEDCHIPLED_0603
- added LED2, LED3, LED4, LED5: GREEN, adafruit:LEDCHIPLED_0603
- added LIGHT_SENSOR_CONNECTOR: (no value), pinhead+:PINHD-2X13SMT
- added R10, R11, R12, R13, R14, R15, R16, R9: 10K, SparkFun-Resistors:RESISTOR0603-RES
- added R17, R18, R19, R20, R21: 330, SparkFun-Resistors:RESISTOR0603
- added SLAVE_LIGHT, SLAVE_TSOP: TEENSY-3.5, teensy-3.5:TEENSY-3.5
- added SW1: (no value), SparkFun-Electromechanical:SW_DIP-8
- added XBEE: XBEE, adafruit:XBEE
- LOGIC_SWITCH, MOTOR_SWITCH, MTR1_OUT, MTR2_OUT, MTR3_OUT, PWR_IN: value (none) -> VH
Connections:
- new net BT_RX: BLUETOOTH.5, MASTER.33/A14/TX5
- new net BT_TX: BLUETOOTH.4, MASTER.34/A15/RX5
- new net DIP1: MASTER.24, R9.1, SW1.8
- new net DIP2: MASTER.25, R10.1, SW1.7
- new net DIP3: MASTER.26, R11.1
- new net DIP4: MASTER.27, R12.1, SW1.5
- new net DIP5: MASTER.28, R13.1, SW1.4
- new net DIP6: MASTER.29/PWM, R14.1, SW1.3
- new net DIP7: MASTER.30/PWM, R15.1, SW1.2
- new net DIP8: MASTER.31/A12/RX4/CS1, R16.1, SW1.1
- new net LED_1: MASTER.50/A24, R18.2, R20.2
- new net LED_2: MASTER.51, R19.2, R21.2
- new net LED_3: MASTER.52
- new net LED_4: MASTER.53
- new net N$22: SW1.6
- new net N$23: LED3.A, R19.1
- new net N$24: LED4.A, R20.1
- new net N$25: LED5.A, R21.1
- new net N$27: LED1.A, R17.1
- new net N$29: LED2.A, R18.1
- new net XBEE_RX: MASTER.48/TX6, XBEE.DIN
- new net XBEE_TX: MASTER.47/RX6, XBEE.DOUT
- net +3V3: now also LIGHT_SENSOR_CONNECTOR.25, R10.2, R11.2, R12.2, R13.2, R14.2, R15.2, R16.2, R9.2, SLAVE_LIGHT.3.3V, SLAVE_TSOP.3.3V, XBEE.VCC; no longer LIGHT_SENSOR.3.3V, TSOP.3.3V
- net +5V: now also R17.2
- net CS_LIGHT_SENSOR: now also SLAVE_LIGHT.10/PWM/TX2/CS0; no longer LIGHT_SENSOR.10/PWM/TX2/CS0
- net CS_TSOP: now also SLAVE_TSOP.15/A1/CS0; no longer TSOP.15/A1/CS0
- net GND: now also LED1.C, LED2.C, LED3.C, LED4.C, LED5.C, LIGHT_SENSOR_CONNECTOR.26, SLAVE_LIGHT.AGND, SLAVE_LIGHT.GND, SLAVE_LIGHT.GND-1, SLAVE_LIGHT.GND-2, SLAVE_LIGHT.GND-3, SLAVE_LIGHT.GND-4, SLAVE_TSOP.AGND, SLAVE_TSOP.GND, SLAVE_TSOP.GND-1, SLAVE_TSOP.GND-2, SLAVE_TSOP.GND-3, SLAVE_TSOP.GND-4, SW1.10, SW1.11, SW1.12, SW1.13, SW1.14, SW1.15, SW1.16, SW1.9, XBEE.GND; no longer LIGHT_SENSOR.AGND, LIGHT_SENSOR.GND, LIGHT_SENSOR.GND-1, LIGHT_SENSOR.GND-2, LIGHT_SENSOR.GND-3, LIGHT_SENSOR.GND-4, TSOP.AGND, TSOP.GND, TSOP.GND-1, TSOP.GND-2, TSOP.GND-3, TSOP.GND-4
- net LS1: now also LIGHT_SENSOR_CONNECTOR.1, SLAVE_LIGHT.14/A0/PWM; no longer LIGHT_SENSOR.14/A0/PWM
- net LS10: now also LIGHT_SENSOR_CONNECTOR.10, SLAVE_LIGHT.23/A9/PWM; no longer LIGHT_SENSOR.23/A9/PWM
- net LS11: now also LIGHT_SENSOR_CONNECTOR.11, SLAVE_LIGHT.A10; no longer LIGHT_SENSOR.A10
- net LS12: now also LIGHT_SENSOR_CONNECTOR.12, SLAVE_LIGHT.A11; no longer LIGHT_SENSOR.A11
- net LS13: now also LIGHT_SENSOR_CONNECTOR.13, SLAVE_LIGHT.31/A12/RX4/CS1; no longer LIGHT_SENSOR.31/A12/RX4/CS1
- net LS14: now also LIGHT_SENSOR_CONNECTOR.14, SLAVE_LIGHT.32/A13/TX4/SCK1; no longer LIGHT_SENSOR.32/A13/TX4/SCK1
- net LS15: now also LIGHT_SENSOR_CONNECTOR.15, SLAVE_LIGHT.33/A14/TX5; no longer LIGHT_SENSOR.33/A14/TX5
- net LS16: now also LIGHT_SENSOR_CONNECTOR.16, SLAVE_LIGHT.34/A15/RX5; no longer LIGHT_SENSOR.34/A15/RX5
- net LS17: now also LIGHT_SENSOR_CONNECTOR.17, SLAVE_LIGHT.35/A16/PWM; no longer LIGHT_SENSOR.35/A16/PWM
- net LS18: now also LIGHT_SENSOR_CONNECTOR.18, SLAVE_LIGHT.36/A17/PWM; no longer LIGHT_SENSOR.36/A17/PWM
- net LS19: now also LIGHT_SENSOR_CONNECTOR.19, SLAVE_LIGHT.37/A18/PWM/SCL1; no longer LIGHT_SENSOR.37/A18/PWM/SCL1
- net LS2: now also LIGHT_SENSOR_CONNECTOR.2, SLAVE_LIGHT.15/A1/CS0; no longer LIGHT_SENSOR.15/A1/CS0
- net LS20: now also LIGHT_SENSOR_CONNECTOR.20, SLAVE_LIGHT.38/A19/PWM/SDA1; no longer LIGHT_SENSOR.38/A19/PWM/SDA1
- net LS21: now also LIGHT_SENSOR_CONNECTOR.21, SLAVE_LIGHT.39/A20; no longer LIGHT_SENSOR.39/A20
- net LS22: now also LIGHT_SENSOR_CONNECTOR.22, SLAVE_LIGHT.A21/DAC0; no longer LIGHT_SENSOR.A21/DAC0
- net LS23: now also LIGHT_SENSOR_CONNECTOR.23, SLAVE_LIGHT.A22/DAC1; no longer LIGHT_SENSOR.A22/DAC1
- net LS24: now also LIGHT_SENSOR_CONNECTOR.24, SLAVE_LIGHT.49/A23; no longer LIGHT_SENSOR.49/A23
- net LS3: now also LIGHT_SENSOR_CONNECTOR.3, SLAVE_LIGHT.16/A2; no longer LIGHT_SENSOR.16/A2
- net LS4: now also LIGHT_SENSOR_CONNECTOR.4, SLAVE_LIGHT.17/A3; no longer LIGHT_SENSOR.17/A3
- net LS5: now also LIGHT_SENSOR_CONNECTOR.5, SLAVE_LIGHT.18/A4/SDA0; no longer LIGHT_SENSOR.18/A4/SDA0
- net LS6: now also LIGHT_SENSOR_CONNECTOR.6, SLAVE_LIGHT.19/A5/SCL0; no longer LIGHT_SENSOR.19/A5/SCL0
- net LS7: now also LIGHT_SENSOR_CONNECTOR.7, SLAVE_LIGHT.20/A6/PWM/CS0; no longer LIGHT_SENSOR.20/A6/PWM/CS0
- net LS8: now also LIGHT_SENSOR_CONNECTOR.8, SLAVE_LIGHT.21/A7/PWM/CS0; no longer LIGHT_SENSOR.21/A7/PWM/CS0
- net LS9: now also LIGHT_SENSOR_CONNECTOR.9, SLAVE_LIGHT.22/A8/PWM; no longer LIGHT_SENSOR.22/A8/PWM
- net MISO: now also SLAVE_LIGHT.12/MISO0, SLAVE_TSOP.12/MISO0; no longer LIGHT_SENSOR.12/MISO0, TSOP.12/MISO0
- net MOSI: now also SLAVE_LIGHT.11/MOSI0, SLAVE_TSOP.11/MOSI0; no longer LIGHT_SENSOR.11/MOSI0, TSOP.11/MOSI0
- net SCK: now also SLAVE_LIGHT.13/SCK0, SLAVE_TSOP.13/SCK0; no longer LIGHT_SENSOR.13/SCK0, TSOP.13/SCK0
- net TEENSY_SCL: now also SLAVE_LIGHT.3/PWM/CAN0TX/SCL2; no longer LIGHT_SENSOR.3/PWM/CAN0TX/SCL2
- net TEENSY_SDA: now also SLAVE_LIGHT.4/PWM/CAN0RX/SDA2, SLAVE_TSOP.38/A19/PWM/SDA1; no longer LIGHT_SENSOR.4/PWM/CAN0RX/SDA2, TSOP.38/A19/PWM/SDA1
- net TEENSY_SDL: now also SLAVE_TSOP.37/A18/PWM/SCL1; no longer TSOP.37/A18/PWM/SCL1
- net TSOP1: now also SLAVE_TSOP.0/RX1/MOSI1; no longer TSOP.0/RX1/MOSI1
- net TSOP10: now also SLAVE_TSOP.9/PWM/RX2/CS0; no longer TSOP.9/PWM/RX2/CS0
- net TSOP11: now also SLAVE_TSOP.10/PWM/TX2/CS0; no longer TSOP.10/PWM/TX2/CS0
- net TSOP12: now also SLAVE_TSOP.14/A0/PWM; no longer TSOP.14/A0/PWM
- net TSOP13: now also SLAVE_TSOP.16/A2; no longer TSOP.16/A2
- net TSOP14: now also SLAVE_TSOP.17/A3; no longer TSOP.17/A3
- net TSOP15: now also SLAVE_TSOP.18/A4/SDA0; no longer TSOP.18/A4/SDA0
- net TSOP16: now also SLAVE_TSOP.19/A5/SCL0; no longer TSOP.19/A5/SCL0
- net TSOP17: now also SLAVE_TSOP.20/A6/PWM/CS0; no longer TSOP.20/A6/PWM/CS0
- net TSOP18: now also SLAVE_TSOP.21/A7/PWM/CS0; no longer TSOP.21/A7/PWM/CS0
- net TSOP19: now also SLAVE_TSOP.22/A8/PWM; no longer TSOP.22/A8/PWM
- net TSOP2: now also SLAVE_TSOP.1/TX1/MISO1; no longer TSOP.1/TX1/MISO1
- net TSOP20: now also SLAVE_TSOP.23/A9/PWM; no longer TSOP.23/A9/PWM
- net TSOP21: now also SLAVE_TSOP.24; no longer TSOP.24
- net TSOP22: now also SLAVE_TSOP.25; no longer TSOP.25
- net TSOP23: now also SLAVE_TSOP.26; no longer TSOP.26
- net TSOP24: now also SLAVE_TSOP.27; no longer TSOP.27
- net TSOP3: now also SLAVE_TSOP.2/PWM; no longer TSOP.2/PWM
- net TSOP4: now also SLAVE_TSOP.3/PWM/CAN0TX/SCL2; no longer TSOP.3/PWM/CAN0TX/SCL2
- net TSOP5: now also SLAVE_TSOP.4/PWM/CAN0RX/SDA2; no longer TSOP.4/PWM/CAN0RX/SDA2
- net TSOP6: now also SLAVE_TSOP.5/PWM; no longer TSOP.5/PWM
- net TSOP7: now also SLAVE_TSOP.6/PWM; no longer TSOP.6/PWM
- net TSOP8: now also SLAVE_TSOP.7/PWM/RX3; no longer TSOP.7/PWM/RX3
- net TSOP9: now also SLAVE_TSOP.8/PWM/TX3; no longer TSOP.8/PWM/TX3
- net TSOP_PWR: now also SLAVE_TSOP.28, SLAVE_TSOP.29/PWM, SLAVE_TSOP.30/PWM, SLAVE_TSOP.31/A12/RX4/CS1; no longer TSOP.28, TSOP.29/PWM, TSOP.30/PWM, TSOP.31/A12/RX4/CS1
Other:
- moved on the sheet: C1, C11, C12, C13, C14, C15, C16, C17, C18, C19, C2, C20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
