File: EAGLE/LJ-STAND/Main.sch (EAGLE design)
At the start: 122 parts, among them Q1 BSS138, Q2 BSS138

Commit message: Eagle stuffs
Parts:
- renumbered TSOP1 to 0, TSOP10 to 17, TSOP11 to 18, TSOP12 to 19, TSOP13 to 20, TSOP14 to 21, TSOP15 to 22, TSOP16 to 23, TSOP17 to 8, TSOP18 to 9, TSOP19 to 10, TSOP2 to 1, TSOP20 to 11, TSOP21 to 12, TSOP22 to 13, TSOP23 to 14, TSOP24 to 15, TSOP3 to 2, TSOP4 to 3, TSOP5 to 4, TSOP6 to 5, TSOP7 to 6, TSOP8 to 7, TSOP9 to 16
Connections:
- removed net LS24: LIGHT_SENSOR_CONNECTOR.24, SLAVE_LIGHT.49/A23
- removed net TSOP24: 15.OUT, SLAVE_TSOP.27
- new net LS0: LIGHT_SENSOR_CONNECTOR.1, SLAVE_LIGHT.14/A0/PWM
- new net TSOP0: 0.OUT, SLAVE_TSOP.0/RX1/MOSI1
- net LS1: now also LIGHT_SENSOR_CONNECTOR.2, SLAVE_LIGHT.15/A1/CS0; no longer LIGHT_SENSOR_CONNECTOR.1, SLAVE_LIGHT.14/A0/PWM
- net LS10: now also LIGHT_SENSOR_CONNECTOR.11, SLAVE_LIGHT.A10; no longer LIGHT_SENSOR_CONNECTOR.10, SLAVE_LIGHT.23/A9/PWM
- net LS11: now also LIGHT_SENSOR_CONNECTOR.12, SLAVE_LIGHT.A11; no longer LIGHT_SENSOR_CONNECTOR.11, SLAVE_LIGHT.A10
- net LS12: now also LIGHT_SENSOR_CONNECTOR.13, SLAVE_LIGHT.31/A12/RX4/CS1; no longer LIGHT_SENSOR_CONNECTOR.12, SLAVE_LIGHT.A11
- net LS13: now also LIGHT_SENSOR_CONNECTOR.14, SLAVE_LIGHT.32/A13/TX4/SCK1; no longer LIGHT_SENSOR_CONNECTOR.13, SLAVE_LIGHT.31/A12/RX4/CS1
- net LS14: now also LIGHT_SENSOR_CONNECTOR.15, SLAVE_LIGHT.33/A14/TX5; no longer LIGHT_SENSOR_CONNECTOR.14, SLAVE_LIGHT.32/A13/TX4/SCK1
- net LS15: now also LIGHT_SENSOR_CONNECTOR.16, SLAVE_LIGHT.34/A15/RX5; no longer LIGHT_SENSOR_CONNECTOR.15, SLAVE_LIGHT.33/A14/TX5
- net LS16: now also LIGHT_SENSOR_CONNECTOR.17, SLAVE_LIGHT.35/A16/PWM; no longer LIGHT_SENSOR_CONNECTOR.16, SLAVE_LIGHT.34/A15/RX5
- net LS17: now also LIGHT_SENSOR_CONNECTOR.18, SLAVE_LIGHT.36/A17/PWM; no longer LIGHT_SENSOR_CONNECTOR.17, SLAVE_LIGHT.35/A16/PWM
- net LS18: now also LIGHT_SENSOR_CONNECTOR.19, SLAVE_LIGHT.37/A18/PWM/SCL1; no longer LIGHT_SENSOR_CONNECTOR.18, SLAVE_LIGHT.36/A17/PWM
- net LS19: now also LIGHT_SENSOR_CONNECTOR.20, SLAVE_LIGHT.38/A19/PWM/SDA1; no longer LIGHT_SENSOR_CONNECTOR.19, SLAVE_LIGHT.37/A18/PWM/SCL1
- net LS2: now also LIGHT_SENSOR_CONNECTOR.3, SLAVE_LIGHT.16/A2; no longer LIGHT_SENSOR_CONNECTOR.2, SLAVE_LIGHT.15/A1/CS0
- net LS20: now also LIGHT_SENSOR_CONNECTOR.21, SLAVE_LIGHT.39/A20; no longer LIGHT_SENSOR_CONNECTOR.20, SLAVE_LIGHT.38/A19/PWM/SDA1
- net LS21: now also LIGHT_SENSOR_CONNECTOR.22, SLAVE_LIGHT.A21/DAC0; no longer LIGHT_SENSOR_CONNECTOR.21, SLAVE_LIGHT.39/A20
- net LS22: now also LIGHT_SENSOR_CONNECTOR.23, SLAVE_LIGHT.A22/DAC1; no longer LIGHT_SENSOR_CONNECTOR.22, SLAVE_LIGHT.A21/DAC0
- net LS23: now also LIGHT_SENSOR_CONNECTOR.24, SLAVE_LIGHT.49/A23; no longer LIGHT_SENSOR_CONNECTOR.23, SLAVE_LIGHT.A22/DAC1
- net LS3: now also LIGHT_SENSOR_CONNECTOR.4, SLAVE_LIGHT.17/A3; no longer LIGHT_SENSOR_CONNECTOR.3, SLAVE_LIGHT.16/A2
- net LS4: now also LIGHT_SENSOR_CONNECTOR.5, SLAVE_LIGHT.18/A4/SDA0; no longer LIGHT_SENSOR_CONNECTOR.4, SLAVE_LIGHT.17/A3
- net LS5: now also LIGHT_SENSOR_CONNECTOR.6, SLAVE_LIGHT.19/A5/SCL0; no longer LIGHT_SENSOR_CONNECTOR.5, SLAVE_LIGHT.18/A4/SDA0
- net LS6: now also LIGHT_SENSOR_CONNECTOR.7, SLAVE_LIGHT.20/A6/PWM/CS0; no longer LIGHT_SENSOR_CONNECTOR.6, SLAVE_LIGHT.19/A5/SCL0
- net LS7: now also LIGHT_SENSOR_CONNECTOR.8, SLAVE_LIGHT.21/A7/PWM/CS0; no longer LIGHT_SENSOR_CONNECTOR.7, SLAVE_LIGHT.20/A6/PWM/CS0
- net LS8: now also LIGHT_SENSOR_CONNECTOR.9, SLAVE_LIGHT.22/A8/PWM; no longer LIGHT_SENSOR_CONNECTOR.8, SLAVE_LIGHT.21/A7/PWM/CS0
- net LS9: now also LIGHT_SENSOR_CONNECTOR.10, SLAVE_LIGHT.23/A9/PWM; no longer LIGHT_SENSOR_CONNECTOR.9, SLAVE_LIGHT.22/A8/PWM
- net TSOP1: now also 1.OUT, SLAVE_TSOP.1/TX1/MISO1; no longer 0.OUT, SLAVE_TSOP.0/RX1/MOSI1
- net TSOP10: now also 10.OUT, SLAVE_TSOP.10/PWM/TX2/CS0; no longer 17.OUT, SLAVE_TSOP.9/PWM/RX2/CS0
- net TSOP11: now also 11.OUT, SLAVE_TSOP.14/A0/PWM; no longer 18.OUT, SLAVE_TSOP.10/PWM/TX2/CS0
- net TSOP12: now also 12.OUT, SLAVE_TSOP.16/A2; no longer 19.OUT, SLAVE_TSOP.14/A0/PWM
- net TSOP13: now also 13.OUT, SLAVE_TSOP.17/A3; no longer 20.OUT, SLAVE_TSOP.16/A2
- net TSOP14: now also 14.OUT, SLAVE_TSOP.18/A4/SDA0; no longer 21.OUT, SLAVE_TSOP.17/A3
- net TSOP15: now also 15.OUT, SLAVE_TSOP.19/A5/SCL0; no longer 22.OUT, SLAVE_TSOP.18/A4/SDA0
- net TSOP16: now also 16.OUT, SLAVE_TSOP.20/A6/PWM/CS0; no longer 23.OUT, SLAVE_TSOP.19/A5/SCL0
- net TSOP17: now also 17.OUT, SLAVE_TSOP.21/A7/PWM/CS0; no longer 8.OUT, SLAVE_TSOP.20/A6/PWM/CS0
- net TSOP18: now also 18.OUT, SLAVE_TSOP.22/A8/PWM; no longer 9.OUT, SLAVE_TSOP.21/A7/PWM/CS0
- net TSOP19: now also 19.OUT, SLAVE_TSOP.23/A9/PWM; no longer 10.OUT, SLAVE_TSOP.22/A8/PWM
- net TSOP2: now also 2.OUT, SLAVE_TSOP.2/PWM; no longer 1.OUT, SLAVE_TSOP.1/TX1/MISO1
- net TSOP20: now also 20.OUT, SLAVE_TSOP.24; no longer 11.OUT, SLAVE_TSOP.23/A9/PWM
- net TSOP21: now also 21.OUT, SLAVE_TSOP.25; no longer 12.OUT, SLAVE_TSOP.24
- net TSOP22: now also 22.OUT, SLAVE_TSOP.26; no longer 13.OUT, SLAVE_TSOP.25
- net TSOP23: now also 23.OUT, SLAVE_TSOP.27; no longer 14.OUT, SLAVE_TSOP.26
- net TSOP3: now also 3.OUT, SLAVE_TSOP.3/PWM/CAN0TX/SCL2; no longer 2.OUT, SLAVE_TSOP.2/PWM
- net TSOP4: now also 4.OUT, SLAVE_TSOP.4/PWM/CAN0RX/SDA2; no longer 3.OUT, SLAVE_TSOP.3/PWM/CAN0TX/SCL2
- net TSOP5: now also 5.OUT, SLAVE_TSOP.5/PWM; no longer 4.OUT, SLAVE_TSOP.4/PWM/CAN0RX/SDA2
- net TSOP6: now also 6.OUT, SLAVE_TSOP.6/PWM; no longer 5.OUT, SLAVE_TSOP.5/PWM
- net TSOP7: now also 7.OUT, SLAVE_TSOP.7/PWM/RX3; no longer 6.OUT, SLAVE_TSOP.6/PWM
- net TSOP8: now also 8.OUT, SLAVE_TSOP.8/PWM/TX3; no longer 7.OUT, SLAVE_TSOP.7/PWM/RX3
- net TSOP9: now also 9.OUT, SLAVE_TSOP.9/PWM/RX2/CS0; no longer 16.OUT, SLAVE_TSOP.8/PWM/TX3

Commit message: Combined I2C & SPI buses into one of each
Parts:
- removed R3, R4: 4.7K, SparkFun-Resistors:RESISTOR0603
Connections:
- net SENSOR_SCL_5V renamed SCL_5V
- net SENSOR_SDA_5V renamed SDA_5V
- removed net PIXY_CS: MASTER.43/CS2, PIXY_SPI.7
- removed net PIXY_MISO: MASTER.45/MISO2, PIXY_SPI.1
- removed net PIXY_MOSI: MASTER.44/MOSI2, PIXY_SPI.4
- removed net PIXY_SCK: MASTER.46/SCK2, PIXY_SPI.3
- removed net SENSOR_SCL: IMU.3, MASTER.19/A5/SCL0, Q1.S, R1.1, R7.1
- removed net SENSOR_SDA: IMU.4, MASTER.18/A4/SDA0, Q2.S, R2.1, R5.1
- removed net TEENSY_SCL: MASTER.37/A18/PWM/SCL1, R3.1, SLAVE_LIGHT.3/PWM/CAN0TX/SCL2
- removed net TEENSY_SDA: MASTER.38/A19/PWM/SDA1, R4.1, SLAVE_LIGHT.4/PWM/CAN0RX/SDA2, SLAVE_TSOP.38/A19/PWM/SDA1
- removed net TEENSY_SDL: SLAVE_TSOP.37/A18/PWM/SCL1
- new net CS_PIXY: MASTER.15/A1/CS0, PIXY_SPI.7
- new net SCL: IMU.3, MASTER.19/A5/SCL0, Q1.S, R1.1, R7.1, SLAVE_LIGHT.3/PWM/CAN0TX/SCL2, SLAVE_TSOP.37/A18/PWM/SCL1
- new net SDA: IMU.4, MASTER.18/A4/SDA0, MASTER.38/A19/PWM/SDA1, Q2.S, R2.1, R5.1, SLAVE_LIGHT.4/PWM/CAN0RX/SDA2, SLAVE_TSOP.38/A19/PWM/SDA1
- net +3V3: no longer R3.2, R4.2
- net MISO: now also PIXY_SPI.1
- net MOSI: now also PIXY_SPI.4
- net SCK: now also PIXY_SPI.3

Commit message: TSOPS placed on pcb and lots of other stuff
Parts:
- removed LED5: GREEN, adafruit:LEDCHIPLED_0603
- added PWR: BLUE, adafruit:LEDCHIPLED_0603
- LED1: value BLUE -> GREEN
- MTR1_OUT, MTR2_OUT, MTR3_OUT: value VH -> PH; device jst-vh:B2P-VH -> adafruit:JST_2PIN-SMT
Connections:
- net GND: now also PWR.C; no longer LED5.C
- net N$23: now also LED2.A; no longer LED3.A
- net N$24: now also LED3.A; no longer LED4.A
- net N$25: now also LED4.A; no longer LED5.A
- net N$27: now also PWR.A; no longer LED1.A
- net N$29: now also LED1.A; no longer LED2.A
Other:
- moved on the sheet: LED1, LED2, LED3, LED4
Changed lines of the file:
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@@
 <part name="GND46" library="supply1" deviceset="GND" device=""/>
 <part name="C24" library="SparkFun-Capacitors" deviceset="CAP" device="0603-CAP" value="0.1uF"/>
-<part name="MTR1_OUT" library="jst-vh" deviceset="B2P-VH" device="" value="VH"/>
+<part name="MTR1_OUT" library="adafruit" deviceset="JST_2PIN" device="-SMT" value="PH"/>
 <part name="C25" library="SparkFun-Capacitors" deviceset="CAP" device="0603-CAP" value="0.01uF"/>
 <part name="C26" library="SparkFun-Capacitors" deviceset="CAP" device="0603-CAP" value="0.22uF"/>
@@
 <part name="GND51" library="supply1" deviceset="GND" device=""/>
 <part name="C29" library="SparkFun-Capacitors" deviceset="CAP" device="0603-CAP" value="0.1uF"/>
-<part name="MTR2_OUT" library="jst-vh" deviceset="B2P-VH" device="" value="VH"/>
+<part name="MTR2_OUT" library="adafruit" deviceset="JST_2PIN" device="-SMT" value="PH"/>
 <part name="C30" library="SparkFun-Capacitors" deviceset="CAP" device="0603-CAP" value="0.01uF"/>
 <part name="C31" library="SparkFun-Capacitors" deviceset="CAP" device="0603-CAP" value="0.22uF"/>
@@
 <part name="GND56" library="supply1" deviceset="GND" device=""/>
 <part name="C34" library="SparkFun-Capacitors" deviceset="CAP" device="0603-CAP" value="0.1uF"/>
-<part name="MTR3_OUT" library="jst-vh" deviceset="B2P-VH" device="" value="VH"/>
+<part name="MTR3_OUT" library="adafruit" deviceset="JST_2PIN" device="-SMT" value="PH"/>
 <part name="C35" library="SparkFun-Capacitors" deviceset="CAP" device="0603-CAP" value="0.01uF"/>
 <part name="C36" library="SparkFun-Capacitors" deviceset="CAP" device="0603-CAP" value="0.22uF"/>
@@
 <part name="+3V21" library="supply1" deviceset="+3V3" device=""/>
 <part name="GND93" library="supply1" deviceset="GND" device=""/>
-<part name="LED1" library="adafruit" deviceset="LED" device="CHIPLED_0603" value="BLUE"/>
+<part name="PWR" library="adafruit" deviceset="LED" device="CHIPLED_0603" value="BLUE"/>
+<part name="LED1" library="adafruit" deviceset="LED" device="CHIPLED_0603" value="GREEN"/>
 <part name="LED2" library="adafruit" deviceset="LED" device="CHIPLED_0603" value="GREEN"/>
-<part name="LED3" library="adafruit" deviceset="LED" device="CHIPLED_0603" value="GREEN"/>
 <part name="XBEE" library="adafruit" deviceset="XBEE" device=""/>
 <part name="GND94" library="supply1" deviceset="GND" device=""/>
@@
 <part name="R18" library="SparkFun-Resistors" deviceset="RESISTOR" device="0603" value="330"/>
 <part name="R19" library="SparkFun-Resistors" deviceset="RESISTOR" device="0603" value="330"/>
+<part name="LED3" library="adafruit" deviceset="LED" device="CHIPLED_0603" value="GREEN"/>
 <part name="LED4" library="adafruit" deviceset="LED" device="CHIPLED_0603" value="GREEN"/>
-<part name="LED5" library="adafruit" deviceset="LED" device="CHIPLED_0603" value="GREEN"/>
 <part name="GND96" library="supply1" deviceset="GND" device=""/>
 <part name="GND99" library="supply1" deviceset="GND" device=""/>
@@
 <instance part="GND46" gate="1" x="177.8" y="309.88"/>
 <instance part="C24" gate="G$1" x="165.1" y="302.26" rot="R90"/>
-<instance part="MTR1_OUT" gate="G$1" x="165.1" y="292.1" rot="R270"/>
+<instance part="MTR1_OUT" gate="G$1" x="162.56" y="289.56" rot="R270"/>
 <instance part="C25" gate="G$1" x="142.24" y="342.9" rot="R180"/>
 <instance part="C26" gate="G$1" x="142.24" y="355.6" rot="R180"/>
@@
 <instance part="GND51" gate="1" x="91.44" y="309.88"/>
 <instance part="C29" gate="G$1" x="78.74" y="302.26" rot="R90"/>
-<instance part="MTR2_OUT" gate="G$1" x="78.74" y="292.1" rot="R270"/>
+<instance part="MTR2_OUT" gate="G$1" x="76.2" y="289.56" rot="R270"/>
 <instance part="C30" gate="G$1" x="55.88" y="342.9" rot="R180"/>
 <instance part="C31" gate="G$1" x="55.88" y="355.6" rot="R180"/>
@@
 <instance part="GND56" gate="1" x="7.62" y="312.42"/>
 <instance part="C34" gate="G$1" x="-5.08" y="304.8" rot="R90"/>
-<instance part="MTR3_OUT" gate="G$1" x="-5.08" y="294.64" rot="R270"/>
+<instance part="MTR3_OUT" gate="G$1" x="-7.62" y="292.1" rot="R270"/>
 <instance part="C35" gate="G$1" x="-27.94" y="345.44" rot="R180"/>
 <instance part="C36" gate="G$1" x="-27.94" y="358.14" rot="R180"/>
@@
 <instance part="+3V21" gate="G$1" x="139.7" y="180.34"/>
 <instance part="GND93" gate="1" x="144.78" y="177.8"/>
-<instance part="LED1" gate="G$1" x="228.6" y="304.8"/>
-<instance part="LED2" gate="G$1" x="243.84" y="304.8"/>
-<instance part="LED3" gate="G$1" x="254" y="304.8"/>
+<instance part="PWR" gate="G$1" x="228.6" y="304.8"/>
+<instance part="LED1" gate="G$1" x="243.84" y="304.8"/>
+<instance part="LED2" gate="G$1" x="254" y="304.8"/>
 <instance part="XBEE" gate="G$1" x="355.6" y="386.08"/>
 <instance part="GND94" gate="1" x="330.2" y="370.84"/>
@@
 <instance part="R18" gate="G$1" x="243.84" y="314.96" rot="R90"/>
 <instance part="R19" gate="G$1" x="254" y="314.96" rot="R90"/>
-<instance part="LED4" gate="G$1" x="264.16" y="304.8"/>
-<instance part="LED5" gate="G$1" x="274.32" y="304.8"/>
+<instance part="LED3" gate="G$1" x="264.16" y="304.8"/>
+<instance part="LED4" gate="G$1" x="274.32" y="304.8"/>
 <instance part="GND96" gate="1" x="264.16" y="294.64"/>
 <instance part="GND99" gate="1" x="274.32" y="294.64"/>
@@
 </segment>
 <segment>
-<pinref part="LED1" gate="G$1" pin="C"/>
+<pinref part="PWR" gate="G$1" pin="C"/>
 <wire x1="228.6" y1="299.72" x2="228.6" y2="297.18" width="0.1524" layer="91"/>
 <pinref part="GND95" gate="1" pin="GND"/>
 </segment>
 <segment>
-<pinref part="LED2" gate="G$1" pin="C"/>
+<pinref part="LED1" gate="G$1" pin="C"/>
 <wire x1="243.84" y1="299.72" x2="243.84" y2="297.18" width="0.1524" layer="91"/>
 <pinref part="GND97" gate="1" pin="GND"/>
 </segment>
 <segment>
-<pinref part="LED3" gate="G$1" pin="C"/>
+<pinref part="LED2" gate="G$1" pin="C"/>
 <wire x1="254" y1="299.72" x2="254" y2="297.18" width="0.1524" layer="91"/>
 <pinref part="GND98" gate="1" pin="GND"/>
 </segment>
 <segment>
-<pinref part="LED4" gate="G$1" pin="C"/>
+<pinref part="LED3" gate="G$1" pin="C"/>
 <wire x1="264.16" y1="299.72" x2="264.16" y2="297.18" width="0.1524" layer="91"/>
 <pinref part="GND96" gate="1" pin="GND"/>
 </segment>
 <segment>
-<pinref part="LED5" gate="G$1" pin="C"/>
+<pinref part="LED4" gate="G$1" pin="C"/>
 <wire x1="274.32" y1="299.72" x2="274.32" y2="297.18" width="0.1524" layer="91"/>
 <pinref part="GND99" gate="1" pin="GND"/>
@@
 <net name="N$27" class="0">
 <segment>
-<pinref part="LED1" gate="G$1" pin="A"/>
+<pinref part="PWR" gate="G$1" pin="A"/>
 <wire x1="228.6" y1="307.34" x2="228.6" y2="309.88" width="0.1524" layer="91"/>
 <pinref part="R17" gate="G$1" pin="1"/>
@@
 <net name="N$29" class="0">
 <segment>
-<pinref part="LED2" gate="G$1" pin="A"/>
+<pinref part="LED1" gate="G$1" pin="A"/>
 <wire x1="243.84" y1="307.34" x2="243.84" y2="309.88" width="0.1524" layer="91"/>
 <pinref part="R18" gate="G$1" pin="1"/>
@@
 <net name="N$23" class="0">
 <segment>
-<pinref part="LED3" gate="G$1" pin="A"/>
+<pinref part="LED2" gate="G$1" pin="A"/>
 <wire x1="254" y1="307.34" x2="254" y2="309.88" width="0.1524" layer="91"/>
 <pinref part="R19" gate="G$1" pin="1"/>
@@
 <net name="N$24" class="0">
 <segment>
-<pinref part="LED4" gate="G$1" pin="A"/>
+<pinref part="LED3" gate="G$1" pin="A"/>
 <wire x1="264.16" y1="307.34" x2="264.16" y2="309.88" width="0.1524" layer="91"/>
 <pinref part="R20" gate="G$1" pin="1"/>
@@
 <net name="N$25" class="0">
 <segment>
-<pinref part="LED5" gate="G$1" pin="A"/>
+<pinref part="LED4" gate="G$1" pin="A"/>
 <wire x1="274.32" y1="307.34" x2="274.32" y2="309.88" width="0.1524" layer="91"/>
 <pinref part="R21" gate="G$1" pin="1"/>

Commit message: PCB Routing
Parts:
- removed XBEE: XBEE, adafruit:XBEE
- renumbered Q1 to SCL, Q2 to SDA
Connections:
- net +3V3: no longer XBEE.VCC
- net GND: no longer XBEE.GND
- net XBEE_RX: no longer XBEE.DIN
- net XBEE_TX: no longer XBEE.DOUT
Changed lines of the file:
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@@
 <part name="MOTOR_FUSE" library="fuse-holder-3568" deviceset="3568-FUSEHOLDER" device="" value="7.5A"/>
 <part name="LOGIC_FUSE" library="fuse-holder-3568" deviceset="3568-FUSEHOLDER" device="" value="2A"/>
-<part name="Q2" library="m-pad-2.1" deviceset="BSS138" device=""/>
+<part name="SDA" library="m-pad-2.1" deviceset="BSS138" device=""/>
 <part name="R5" library="SparkFun-Resistors" deviceset="RESISTOR" device="0603-RES" value="10K"/>
 <part name="R6" library="SparkFun-Resistors" deviceset="RESISTOR" device="0603-RES" value="10K"/>
 <part name="+3V10" library="supply1" deviceset="+3V3" device=""/>
 <part name="P+4" library="supply1" deviceset="+5V" device=""/>
-<part name="Q1" library="m-pad-2.1" deviceset="BSS138" device=""/>
+<part name="SCL" library="m-pad-2.1" deviceset="BSS138" device=""/>
 <part name="R7" library="SparkFun-Resistors" deviceset="RESISTOR" device="0603-RES" value="10K"/>
 <part name="R8" library="SparkFun-Resistors" deviceset="RESISTOR" device="0603-RES" value="10K"/>
@@
 <part name="LED1" library="adafruit" deviceset="LED" device="CHIPLED_0603" value="GREEN"/>
 <part name="LED2" library="adafruit" deviceset="LED" device="CHIPLED_0603" value="GREEN"/>
-<part name="XBEE" library="adafruit" deviceset="XBEE" device=""/>
 <part name="GND94" library="supply1" deviceset="GND" device=""/>
 <part name="+3V22" library="supply1" deviceset="+3V3" device=""/>
@@
 <instance part="MOTOR_FUSE" gate="G$1" x="-12.7" y="129.54"/>
 <instance part="LOGIC_FUSE" gate="G$1" x="-12.7" y="111.76"/>
-<instance part="Q2" gate="G$1" x="50.8" y="236.22" rot="R270"/>
+<instance part="SDA" gate="G$1" x="50.8" y="236.22" rot="R270"/>
 <instance part="R5" gate="G$1" x="43.18" y="241.3" rot="R90"/>
 <instance part="R6" gate="G$1" x="58.42" y="241.3" rot="R90"/>
 <instance part="+3V10" gate="G$1" x="43.18" y="254"/>
 <instance part="P+4" gate="1" x="58.42" y="254"/>
-<instance part="Q1" gate="G$1" x="50.8" y="198.12" rot="R270"/>
+<instance part="SCL" gate="G$1" x="50.8" y="198.12" rot="R270"/>
 <instance part="R7" gate="G$1" x="43.18" y="203.2" rot="R90"/>
 <instance part="R8" gate="G$1" x="58.42" y="203.2" rot="R90"/>
@@
 <instance part="LED1" gate="G$1" x="243.84" y="304.8"/>
 <instance part="LED2" gate="G$1" x="254" y="304.8"/>
-<instance part="XBEE" gate="G$1" x="355.6" y="386.08"/>
 <instance part="GND94" gate="1" x="330.2" y="370.84"/>
 <instance part="+3V22" gate="G$1" x="330.2" y="401.32"/>
@@
 </segment>
 <segment>
-<pinref part="XBEE" gate="G$1" pin="GND"/>
 <wire x1="332.74" y1="373.38" x2="330.2" y2="373.38" width="0.1524" layer="91"/>
 <pinref part="GND94" gate="1" pin="GND"/>
@@
 <wire x1="43.18" y1="246.38" x2="43.18" y2="248.92" width="0.1524" layer="91"/>
 <wire x1="43.18" y1="251.46" x2="43.18" y2="248.92" width="0.1524" layer="91"/>
-<pinref part="Q2" gate="G$1" pin="G"/>
+<pinref part="SDA" gate="G$1" pin="G"/>
 <wire x1="43.18" y1="248.92" x2="48.26" y2="248.92" width="0.1524" layer="91"/>
 <wire x1="48.26" y1="248.92" x2="48.26" y2="241.3" width="0.1524" layer="91"/>
@@
 <wire x1="43.18" y1="208.28" x2="43.18" y2="210.82" width="0.1524" layer="91"/>
 <wire x1="43.18" y1="213.36" x2="43.18" y2="210.82" width="0.1524" layer="91"/>
-<pinref part="Q1" gate="G$1" pin="G"/>
+<pinref part="SCL" gate="G$1" pin="G"/>
 <wire x1="43.18" y1="210.82" x2="48.26" y2="210.82" width="0.1524" layer="91"/>
 <wire x1="48.26" y1="210.82" x2="48.26" y2="203.2" width="0.1524" layer="91"/>
@@
 </segment>
 <segment>
-<pinref part="XBEE" gate="G$1" pin="VCC"/>
 <pinref part="+3V22" gate="G$1" pin="+3V3"/>
 <wire x1="332.74" y1="396.24" x2="330.2" y2="396.24" width="0.1524" layer="91"/>
@@
 </segment>
 <segment>
-<pinref part="XBEE" gate="G$1" pin="DOUT"/>
 <wire x1="332.74" y1="393.7" x2="330.2" y2="393.7" width="0.1524" layer="91"/>
 <label x="330.2" y="393.7" size="1.778" layer="95" rot="R180" xref="yes"/>
@@
 </segment>
 <segment>
-<pinref part="XBEE" gate="G$1" pin="DIN"/>
 <wire x1="332.74" y1="391.16" x2="330.2" y2="388.62" width="0.1524" layer="91"/>
 <label x="330.2" y="388.62" size="1.778" layer="95" rot="R180" xref="yes"/>
@@
 </segment>
 <segment>
-<pinref part="Q2" gate="G$1" pin="S"/>
+<pinref part="SDA" gate="G$1" pin="S"/>
 <wire x1="45.72" y1="233.68" x2="43.18" y2="233.68" width="0.1524" layer="91"/>
 <wire x1="43.18" y1="233.68" x2="43.18" y2="236.22" width="0.1524" layer="91"/>
@@
 </segment>
 <segment>
-<pinref part="Q1" gate="G$1" pin="S"/>
+<pinref part="SCL" gate="G$1" pin="S"/>
 <wire x1="45.72" y1="195.58" x2="43.18" y2="195.58" width="0.1524" layer="91"/>
 <wire x1="43.18" y1="195.58" x2="43.18" y2="198.12" width="0.1524" layer="91"/>
@@
 <net name="SCL_5V" class="0">
 <segment>
-<pinref part="Q1" gate="G$1" pin="D"/>
+<pinref part="SCL" gate="G$1" pin="D"/>
 <wire x1="55.88" y1="195.58" x2="58.42" y2="195.58" width="0.1524" layer="91"/>
 <pinref part="R8" gate="G$1" pin="1"/>
@@
 <net name="SDA_5V" class="0">
 <segment>
-<pinref part="Q2" gate="G$1" pin="D"/>
+<pinref part="SDA" gate="G$1" pin="D"/>
 <wire x1="55.88" y1="233.68" x2="58.42" y2="233.68" width="0.1524" layer="91"/>
 <pinref part="R6" gate="G$1" pin="1"/>
