File: EAGLE/LJ-STAND/Main.sch (EAGLE design)
At the start: 129 parts

Commit message: Main pcb
Parts:
- removed MTR1_OUT_RIGHT, MTR2_OUT_LEFT, MTR3_OUT_BACKRIGHT, MTR4_OUT_BACKLEFT: PH, adafruit:JST_2PIN-SMT
- added BACKLEFT, BACKRIGHT, LEFT, RIGHT: PH, adafruit:JST_2PIN-THM
- added SONAR: (no value), SparkFun-Connectors:M04PTH
- C14: value 10uF Tantalum -> 10uF
- LIGHT_GATE: device SparkFun-Connectors:M04PTH -> SparkFun-Connectors:M05PTH
Connections:
- net +5V: now also SONAR.1
- net GND: now also LIGHT_GATE.5, SONAR.4
- net N$1: now also LEFT.2; no longer MTR2_OUT_LEFT.2
- net N$14: now also BACKRIGHT.2; no longer MTR3_OUT_BACKRIGHT.2
- net N$16: now also BACKRIGHT.1; no longer MTR3_OUT_BACKRIGHT.1
- net N$2: now also LEFT.1; no longer MTR2_OUT_LEFT.1
- net N$22: now also BACKLEFT.2; no longer MTR4_OUT_BACKLEFT.2
- net N$26: now also BACKLEFT.1; no longer MTR4_OUT_BACKLEFT.1
- net N$5: now also RIGHT.2; no longer MTR1_OUT_RIGHT.2
- net N$7: now also RIGHT.1; no longer MTR1_OUT_RIGHT.1
- net SCL_5V: now also SONAR.3
- net SDA_5V: now also SONAR.2

Commit message: Main pcb
Connections:
- removed net N$37: LIGHT_GATE.1
- net +5V: now also LIGHT_GATE.1
Changed lines of the file:
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@@
 <part name="D1" library="diode" deviceset="SCHOTTKY-DIODE" device="P6T15"/>
 <part name="D2" library="adafruit" deviceset="DIODE" device="_SOD-123FL"/>
-<part name="P+7" library="supply1" deviceset="+5V" device=""/>
 <part name="GND94" library="supply1" deviceset="GND" device=""/>
 <part name="+3V8" library="supply1" deviceset="+3V3" device=""/>
@@
 <part name="GND106" library="supply1" deviceset="GND" device=""/>
 <part name="P+8" library="supply1" deviceset="+5V" device=""/>
+<part name="P+7" library="supply1" deviceset="+5V" device=""/>
 </parts>
 <sheets>
@@
 <instance part="D1" gate="G$1" x="-30.48" y="124.46"/>
 <instance part="D2" gate="G$1" x="55.88" y="114.3"/>
-<instance part="P+7" gate="1" x="261.62" y="259.08"/>
 <instance part="GND94" gate="1" x="264.16" y="233.68"/>
 <instance part="+3V8" gate="G$1" x="254" y="256.54"/>
@@
 <instance part="GND106" gate="1" x="139.7" y="149.86"/>
 <instance part="P+8" gate="1" x="139.7" y="167.64"/>
+<instance part="P+7" gate="1" x="261.62" y="259.08"/>
 </instances>
 <busses>
@@
 <wire x1="139.7" y1="162.56" x2="139.7" y2="165.1" width="0.1524" layer="91"/>
 <pinref part="P+8" gate="1" pin="+5V"/>
+</segment>
+<segment>
+<wire x1="266.7" y1="254" x2="261.62" y2="254" width="0.1524" layer="91"/>
+<wire x1="261.62" y1="254" x2="261.62" y2="256.54" width="0.1524" layer="91"/>
+<pinref part="LIGHT_GATE" gate="G$1" pin="1"/>
+<pinref part="P+7" gate="1" pin="+5V"/>
 </segment>
 </net>
@@
 </segment>
 </net>
-<net name="N$37" class="0">
-<segment>
-<wire x1="266.7" y1="254" x2="261.62" y2="254" width="0.1524" layer="91"/>
-<wire x1="261.62" y1="254" x2="261.62" y2="256.54" width="0.1524" layer="91"/>
-<pinref part="P+7" gate="1" pin="+5V"/>
-<pinref part="LIGHT_GATE" gate="G$1" pin="1"/>
-</segment>
-</net>

Commit message: PCB finalising
Parts:
- C11, C13: device SparkFun-Capacitors:CAP0603-CAP -> SparkFun-Capacitors:CAP0805
Changed lines of the file:
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@@
 <part name="VREG-5V" library="V78-2000-switching-regulator" deviceset="V78-2000" device=""/>
 <part name="GND8" library="supply1" deviceset="GND" device=""/>
-<part name="C11" library="SparkFun-Capacitors" deviceset="CAP" device="0603-CAP" value="10uF"/>
+<part name="C11" library="SparkFun-Capacitors" deviceset="CAP" device="0805" value="10uF"/>
 <part name="C12" library="SparkFun-Capacitors" deviceset="CAP" device="0805" value="22uF"/>
 <part name="P+1" library="supply1" deviceset="+5V" device=""/>
@@
 <part name="+3V1" library="supply1" deviceset="+3V3" device=""/>
 <part name="PWR_IN" library="jst-vh" deviceset="B2P-VH" device="" value="VH"/>
-<part name="C13" library="SparkFun-Capacitors" deviceset="CAP" device="0603-CAP" value="10uF"/>
+<part name="C13" library="SparkFun-Capacitors" deviceset="CAP" device="0805" value="10uF"/>
 <part name="C14" library="SparkFun-Capacitors" deviceset="CAP" device="0805" value="10uF"/>
 <part name="MOTOR_SWITCH" library="jst-vh" deviceset="B2P-VH" device="" value="VH"/>
