File: EAGLE/LJ-STAND/Light Sensor.sch (EAGLE design)
At the start: 2 parts

Commit message: Light sensor connector
Connections:
- net N$1 renamed LS0
- net N$2 renamed LS1
- net N$3 renamed LS2
- net N$4 renamed LS3
- net N$5 renamed LS5
- net N$6 renamed LS7
- net N$7 renamed LS9
- net N$8 renamed LS11
- new net +3V3: JP1.25
- new net LS10: JP1.11
- new net LS12: JP1.13, JP1.14
- new net LS13: JP1.16
- new net LS14: JP1.15
- new net LS15: JP1.18
- new net LS16: JP1.17
- new net LS17: JP1.20
- new net LS18: JP1.19, JP1.22
- new net LS20: JP1.21, JP1.24
- new net LS22: JP1.23
- new net LS4: JP1.5
- new net LS6: JP1.7
- new net LS8: JP1.9
- net GND: now also JP1.26
Changed lines of the file:
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@@
 <?xml version="1.0" encoding="utf-8"?>
 <!DOCTYPE eagle SYSTEM "eagle.dtd">
-<eagle version="7.2.0">
+<eagle version="7.5.0">
 <drawing>
 <settings>
@@
 <part name="GND1" library="m-pad-2.1" deviceset="GND1" device=""/>
 <part name="JP1" library="pinhead+" deviceset="PINHD-2X13" device="SMT"/>
+<part name="+3V1" library="supply1" deviceset="+3V3" device=""/>
+<part name="GND2" library="supply1" deviceset="GND" device=""/>
 </parts>
 <sheets>
@@
 <instance part="GND1" gate="1" x="17.78" y="48.26"/>
 <instance part="JP1" gate="A" x="93.98" y="99.06"/>
+<instance part="+3V1" gate="G$1" x="68.58" y="88.9"/>
+<instance part="GND2" gate="1" x="106.68" y="81.28"/>
 </instances>
 <busses>
@@
 <pinref part="GND1" gate="1" pin="GND"/>
 </segment>
-</net>
-<net name="N$1" class="0">
+<segment>
+<pinref part="JP1" gate="A" pin="26"/>
+<wire x1="99.06" y1="83.82" x2="106.68" y2="83.82" width="0.1524" layer="91"/>
+<pinref part="GND2" gate="1" pin="GND"/>
+</segment>
+</net>
+<net name="LS0" class="0">
 <segment>
 <pinref part="JP1" gate="A" pin="1"/>
 <wire x1="91.44" y1="114.3" x2="83.82" y2="114.3" width="0.1524" layer="91"/>
-</segment>
-</net>
-<net name="N$2" class="0">
+<label x="83.82" y="114.3" size="1.778" layer="95" rot="R180" xref="yes"/>
+</segment>
+</net>
+<net name="LS1" class="0">
 <segment>
 <pinref part="JP1" gate="A" pin="2"/>
 <wire x1="99.06" y1="114.3" x2="106.68" y2="114.3" width="0.1524" layer="91"/>
-</segment>
-</net>
-<net name="N$3" class="0">
+<label x="106.68" y="114.3" size="1.778" layer="95" xref="yes"/>
+</segment>
+</net>
+<net name="LS2" class="0">
 <segment>
 <pinref part="JP1" gate="A" pin="3"/>
 <wire x1="91.44" y1="111.76" x2="83.82" y2="111.76" width="0.1524" layer="91"/>
-</segment>
-</net>
-<net name="N$4" class="0">
+<label x="83.82" y="111.76" size="1.778" layer="95" rot="R180" xref="yes"/>
+</segment>
+</net>
+<net name="LS3" class="0">
 <segment>
 <pinref part="JP1" gate="A" pin="4"/>
 <wire x1="99.06" y1="111.76" x2="106.68" y2="111.76" width="0.1524" layer="91"/>
-</segment>
-</net>
-<net name="N$5" class="0">
+<label x="106.68" y="111.76" size="1.778" layer="95" xref="yes"/>
+</segment>
+</net>
+<net name="LS5" class="0">
 <segment>
 <pinref part="JP1" gate="A" pin="6"/>
 <wire x1="99.06" y1="109.22" x2="106.68" y2="109.22" width="0.1524" layer="91"/>
-</segment>
-</net>
-<net name="N$6" class="0">
+<label x="106.68" y="109.22" size="1.778" layer="95" xref="yes"/>
+</segment>
+</net>
+<net name="LS7" class="0">
 <segment>
 <pinref part="JP1" gate="A" pin="8"/>
 <wire x1="99.06" y1="106.68" x2="106.68" y2="106.68" width="0.1524" layer="91"/>
-</segment>
-</net>
-<net name="N$7" class="0">
+<label x="106.68" y="106.68" size="1.778" layer="95" xref="yes"/>
+</segment>
+</net>
+<net name="LS9" class="0">
 <segment>
 <pinref part="JP1" gate="A" pin="10"/>
 <wire x1="99.06" y1="104.14" x2="106.68" y2="104.14" width="0.1524" layer="91"/>
-</segment>
-</net>
-<net name="N$8" class="0">
+<label x="106.68" y="104.14" size="1.778" layer="95" xref="yes"/>
+</segment>
+</net>
+<net name="LS11" class="0">
 <segment>
 <pinref part="JP1" gate="A" pin="12"/>
 <wire x1="99.06" y1="101.6" x2="106.68" y2="101.6" width="0.1524" layer="91"/>
-</segment>
-</net>
+<label x="106.68" y="101.6" size="1.778" layer="95" xref="yes"/>
+</segment>
+</net>
+<net name="LS4" class="0">
+<segment>
+<pinref part="JP1" gate="A" pin="5"/>
+<wire x1="91.44" y1="109.22" x2="83.82" y2="109.22" width="0.1524" layer="91"/>
+<label x="83.82" y="109.22" size="1.778" layer="95" rot="R180" xref="yes"/>
+</segment>
+</net>
+<net name="LS6" class="0">
+<segment>
+<pinref part="JP1" gate="A" pin="7"/>
+<wire x1="91.44" y1="106.68" x2="83.82" y2="106.68" width="0.1524" layer="91"/>
+<label x="83.82" y="106.68" size="1.778" layer="95" rot="R180" xref="yes"/>
+</segment>
+</net>
+<net name="LS8" class="0">
+<segment>
+<pinref part="JP1" gate="A" pin="9"/>
+<wire x1="91.44" y1="104.14" x2="83.82" y2="104.14" width="0.1524" layer="91"/>
+<label x="83.82" y="104.14" size="1.778" layer="95" rot="R180" xref="yes"/>
+</segment>
+</net>
+<net name="LS10" class="0">
+<segment>
+<pinref part="JP1" gate="A" pin="11"/>
+<wire x1="91.44" y1="101.6" x2="83.82" y2="101.6" width="0.1524" layer="91"/>
+<label x="83.82" y="101.6" size="1.778" layer="95" rot="R180" xref="yes"/>
+</segment>
+</net>
+<net name="LS12" class="0">
+<segment>
+<pinref part="JP1" gate="A" pin="13"/>
+<wire x1="91.44" y1="99.06" x2="83.82" y2="99.06" width="0.1524" layer="91"/>
+<label x="83.82" y="99.06" size="1.778" layer="95" rot="R180" xref="yes"/>
+</segment>
+<segment>
+<pinref part="JP1" gate="A" pin="14"/>
+<wire x1="99.06" y1="99.06" x2="106.68" y2="99.06" width="0.1524" layer="91"/>
+<label x="106.68" y="99.06" size="1.778" layer="95" xref="yes"/>
+</segment>
+</net>
+<net name="LS14" class="0">
+<segment>
+<pinref part="JP1" gate="A" pin="15"/>
+<wire x1="91.44" y1="96.52" x2="83.82" y2="96.52" width="0.1524" layer="91"/>
+<label x="83.82" y="96.52" size="1.778" layer="95" rot="R180" xref="yes"/>
+</segment>
+</net>
+<net name="LS16" class="0">
+<segment>
+<pinref part="JP1" gate="A" pin="17"/>
+<wire x1="91.44" y1="93.98" x2="83.82" y2="93.98" width="0.1524" layer="91"/>
+<label x="83.82" y="93.98" size="1.778" layer="95" rot="R180" xref="yes"/>
+</segment>
+</net>
+<net name="LS18" class="0">
+<segment>
+<pinref part="JP1" gate="A" pin="19"/>
+<wire x1="91.44" y1="91.44" x2="83.82" y2="91.44" width="0.1524" layer="91"/>
+<label x="83.82" y="91.44" size="1.778" layer="95" rot="R180" xref="yes"/>
+</segment>
+<segment>
+<pinref part="JP1" gate="A" pin="22"/>
+<wire x1="99.06" y1="88.9" x2="106.68" y2="88.9" width="0.1524" layer="91"/>
+<label x="106.68" y="88.9" size="1.778" layer="95" xref="yes"/>
+</segment>
+</net>
+<net name="LS20" class="0">
+<segment>
+<pinref part="JP1" gate="A" pin="21"/>
+<wire x1="91.44" y1="88.9" x2="83.82" y2="88.9" width="0.1524" layer="91"/>
+<label x="83.82" y="88.9" size="1.778" layer="95" rot="R180" xref="yes"/>
+</segment>
+<segment>
+<pinref part="JP1" gate="A" pin="24"/>
+<wire x1="99.06" y1="86.36" x2="106.68" y2="86.36" width="0.1524" layer="91"/>
+<label x="106.68" y="86.36" size="1.778" layer="95" xref="yes"/>
+</segment>
+</net>
+<net name="LS22" class="0">
+<segment>
+<pinref part="JP1" gate="A" pin="23"/>
+<wire x1="91.44" y1="86.36" x2="83.82" y2="86.36" width="0.1524" layer="91"/>
+<label x="83.82" y="86.36" size="1.778" layer="95" rot="R180" xref="yes"/>
+</segment>
+</net>
+<net name="LS13" class="0">
+<segment>
+<pinref part="JP1" gate="A" pin="16"/>
+<wire x1="99.06" y1="96.52" x2="106.68" y2="96.52" width="0.1524" layer="91"/>
+<label x="106.68" y="96.52" size="1.778" layer="95" xref="yes"/>
+</segment>
+</net>
+<net name="LS15" class="0">
+<segment>
+<pinref part="JP1" gate="A" pin="18"/>
+<wire x1="99.06" y1="93.98" x2="106.68" y2="93.98" width="0.1524" layer="91"/>
+<label x="106.68" y="93.98" size="1.778" layer="95" xref="yes"/>
+</segment>
+</net>
+<net name="LS17" class="0">
+<segment>
+<pinref part="JP1" gate="A" pin="20"/>
+<wire x1="99.06" y1="91.44" x2="106.68" y2="91.44" width="0.1524" layer="91"/>
+<label x="106.68" y="91.44" size="1.778" layer="95" xref="yes"/>
+</segment>
+</net>
+<net name="+3V3" class="0">
+<segment>
+<pinref part="JP1" gate="A" pin="25"/>
+<wire x1="91.44" y1="83.82" x2="68.58" y2="83.82" width="0.1524" layer="91"/>
+<wire x1="68.58" y1="83.82" x2="68.58" y2="86.36" width="0.1524" layer="91"/>
+<pinref part="+3V1" gate="G$1" pin="+3V3"/>
+</segment>
+</net>

Commit message: Trimpot on light pcb
Parts:
- added R1: (no value), rcl:R-TRIMM3296W
- added R2: 100, SparkFun-Resistors:RESISTOR0603
- renumbered JP1 to LIGHT_SENSOR_CONNECTOR
Connections:
- new net LED_PWR: R1.S, R2.2
- new net N$1: LED1.A, R2.1
- net +3V3: now also R1.A
