File: EAGLE/LJ-STAND/Light Sensor.sch (EAGLE design)
At the start: 122 parts

Commit message: changed 0805 to 0603 leds
Parts:
- LED0, LED1, LED10, LED11, LED12, LED13, LED14, LED15, LED16, LED17, LED18, LED19, LED2, LED20, LED21, LED22, LED23, LED3, LED4, LED5, LED6, LED7, LED8, LED9: device adafruit:LEDCHIP-LED0805 -> adafruit:LEDCHIP-LED0603
