File: EAGLE/LJ-STAND/Kicker.brd (EAGLE design)
At the start: 160 x 100 mm, 10 parts, among them K1 G5LE, Q1 BSS92

Commit message: Hexagon too small
Parts:
- added HVIN, HVOUT: (no value), jst-vh:B2P-VH
- added R3, R4: (no value), SparkFun-Resistors:AXIAL-0.8
- moved SIGNAL 216.0 mm to (110.2, -127.2)
- moved Q1 209.4 mm to (119.0, -118.1)
- moved KICKER_PWR 190.9 mm to (81.3, -123.2)
- moved R1 188.2 mm to (103.3, -101.7)
- moved SOLENOID_OUT 186.3 mm to (118.9, -92.4)
- moved K1 180.7 mm to (131.1, -111.1), turned to 90 degrees
- moved R2 180.5 mm to (103.0, -105.0), turned to 180 degrees
- moved D1 137.4 mm to (104.5, -119.5)
- moved D2 135.1 mm to (104.6, -124.3)
- moved C1 108.7 mm to (85.0, -97.9), turned to 90 degrees
Connections:
- new net HV: HVOUT.1, R4.P$2
- new net N$1: K1.O, R4.P$1
- new net N$4: HVOUT.2
- new net N$7: HVIN.2
- net GND: now also R3.P$1
- net N$5: now also R3.P$2
- net VCC: now also HVIN.1; no longer K1.O
Other:
- board size 160 x 100 mm -> 43 x 49 mm

Commit message: Kicker pcb - from a few days ago
Parts:
- added D3: 1N4004, diode:DO41-10
- Q1: value BSS92 -> BSS296
- R1: value 1K -> 50
- R3: value (none) -> 56K; device SparkFun-Resistors:AXIAL-0.8 -> SparkFun-Resistors:AXIAL-0.3
- R4: value (none) -> 50; device SparkFun-Resistors:AXIAL-0.8 -> SparkFun-Resistors:AXIAL-0.1
- moved R3 59.1 mm to (123.7, -95.1), turned to 270 degrees
- moved R4 48.1 mm to (110.3, -125.1), turned to 270 degrees
- moved KICKER_PWR 36.3 mm to (117.1, -117.0)
- moved HVOUT 34.9 mm to (117.9, -94.5)
- moved R1 34.6 mm to (135.8, -113.7), flipped to the bottom
- moved R2 33.3 mm to (135.8, -110.8), flipped to the bottom
- moved SIGNAL 31.0 mm to (108.9, -96.3)
- moved HVIN 28.4 mm to (102.2, -104.0), turned to 90 degrees
- moved C1 24.6 mm to (101.4, -116.3)
- moved D1 17.3 mm to (119.2, -128.6)
- moved D2 14.7 mm to (119.2, -125.5)
- moved Q1 14.6 mm to (119.0, -132.7), turned to 180 degrees
- moved SOLENOID_OUT 13.9 mm to (117.0, -106.2)
- moved K1 0.20 mm to (130.9, -111.1)
Connections:
- removed net N$7: HVIN.2
- net GND: now also HVIN.2, HVOUT.2
- net HV: now also D3.C; no longer HVOUT.1
- net N$4: now also D3.A, HVIN.1; no longer HVOUT.2
- net VCC: now also HVOUT.1; no longer HVIN.1
