File: EAGLE/LJ-STAND/Kicker.sch (EAGLE design)
At the start: 14 parts, among them K1 G5LE, Q1 BSS92

Commit message: Kicker pcb - from a few days ago
Parts:
- added D3: 1N4004, diode:1N4004
- Q1: value BSS92 -> BSS296; device transistor-fet:BSS92 -> transistor-fet:BSS296
- R1: value 1K -> 50
- R3: value (none) -> 56K; device SparkFun-Resistors:RESISTORPTH-2W -> SparkFun-Resistors:100KOHM-1/4W-1%(PTH)HORIZ
- R4: value (none) -> 50; device SparkFun-Resistors:RESISTORPTH-2W -> SparkFun-Resistors:RESISTORPTH-1/4W-VERT
Connections:
- removed net N$7: HVIN.2
- net GND: now also HVIN.2, HVOUT.2
- net HV: now also D3.C; no longer HVOUT.1
- net N$4: now also D3.A, HVIN.1; no longer HVOUT.2
- net VCC: now also HVOUT.1; no longer HVIN.1
Other:
- moved on the sheet: R3
Changed lines of the file:
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@@
 <part name="GND1" library="supply1" deviceset="GND" device=""/>
 <part name="SIGNAL" library="jst-ph" deviceset="B2B-PH-*" device="K-S"/>
-<part name="R1" library="SparkFun-Resistors" deviceset="RESISTOR" device="0603" value="1K"/>
+<part name="R1" library="SparkFun-Resistors" deviceset="RESISTOR" device="0603" value="50"/>
 <part name="GND2" library="supply1" deviceset="GND" device=""/>
-<part name="Q1" library="transistor-fet" deviceset="BSS92" device=""/>
+<part name="Q1" library="transistor-fet" deviceset="BSS296" device=""/>
 <part name="R2" library="SparkFun-Resistors" deviceset="RESISTOR" device="0805-RES" value="100K"/>
 <part name="K1" library="relay" deviceset="G5LE" device=""/>
@@
 <part name="D1" library="diode" deviceset="1N4004" device=""/>
 <part name="D2" library="diode" deviceset="1N4004" device=""/>
-<part name="R3" library="SparkFun-Resistors" deviceset="RESISTOR" device="PTH-2W"/>
+<part name="R3" library="SparkFun-Resistors" deviceset="100KOHM-1/4W-1%(PTH)" device="HORIZ" value="56K"/>
 <part name="GND5" library="supply1" deviceset="GND" device=""/>
 <part name="HVIN" library="jst-vh" deviceset="B2P-VH" device=""/>
 <part name="HVOUT" library="jst-vh" deviceset="B2P-VH" device=""/>
-<part name="R4" library="SparkFun-Resistors" deviceset="RESISTOR" device="PTH-2W"/>
+<part name="R4" library="SparkFun-Resistors" deviceset="RESISTOR" device="PTH-1/4W-VERT" value="50"/>
+<part name="GND6" library="supply1" deviceset="GND" device=""/>
+<part name="GND7" library="supply1" deviceset="GND" device=""/>
+<part name="D3" library="diode" deviceset="1N4004" device=""/>
 </parts>
 <sheets>
@@
 <instance part="D1" gate="1" x="68.58" y="127" rot="R90"/>
 <instance part="D2" gate="1" x="93.98" y="114.3" rot="R90"/>
-<instance part="R3" gate="G$1" x="119.38" y="132.08" rot="R90"/>
-<instance part="GND5" gate="1" x="114.3" y="124.46"/>
+<instance part="R3" gate="G$1" x="109.22" y="139.7" rot="R180"/>
+<instance part="GND5" gate="1" x="116.84" y="137.16"/>
 <instance part="HVIN" gate="G$1" x="12.7" y="119.38"/>
 <instance part="HVOUT" gate="G$1" x="12.7" y="132.08"/>
 <instance part="R4" gate="G$1" x="86.36" y="139.7" rot="R90"/>
+<instance part="GND6" gate="1" x="5.08" y="127"/>
+<instance part="GND7" gate="1" x="5.08" y="114.3"/>
+<instance part="D3" gate="1" x="2.54" y="119.38" rot="R180"/>
 </instances>
 <busses>
@@
 <pinref part="R3" gate="G$1" pin="1"/>
 <pinref part="GND5" gate="1" pin="GND"/>
-<wire x1="119.38" y1="127" x2="114.3" y2="127" width="0.1524" layer="91"/>
+<wire x1="114.3" y1="139.7" x2="116.84" y2="139.7" width="0.1524" layer="91"/>
+</segment>
+<segment>
+<pinref part="HVIN" gate="G$1" pin="2"/>
+<wire x1="12.7" y1="116.84" x2="5.08" y2="116.84" width="0.1524" layer="91"/>
+<pinref part="GND7" gate="1" pin="GND"/>
+</segment>
+<segment>
+<pinref part="HVOUT" gate="G$1" pin="2"/>
+<wire x1="12.7" y1="129.54" x2="5.08" y2="129.54" width="0.1524" layer="91"/>
+<pinref part="GND6" gate="1" pin="GND"/>
 </segment>
 </net>
@@
 <pinref part="C1" gate="G$1" pin="+"/>
 <wire x1="101.6" y1="137.16" x2="101.6" y2="139.7" width="0.1524" layer="91"/>
-<wire x1="101.6" y1="139.7" x2="114.3" y2="139.7" width="0.1524" layer="91"/>
+<pinref part="R3" gate="G$1" pin="2"/>
+<wire x1="101.6" y1="139.7" x2="104.14" y2="139.7" width="0.1524" layer="91"/>
 <junction x="101.6" y="139.7"/>
-<wire x1="114.3" y1="139.7" x2="119.38" y2="137.16" width="0.1524" layer="91"/>
-<pinref part="R3" gate="G$1" pin="2"/>
 </segment>
 </net>
@@
 </segment>
 <segment>
-<pinref part="HVIN" gate="G$1" pin="1"/>
-<wire x1="12.7" y1="119.38" x2="7.62" y2="119.38" width="0.1524" layer="91"/>
-<label x="7.62" y="119.38" size="1.778" layer="95" rot="R180" xref="yes"/>
+<pinref part="HVOUT" gate="G$1" pin="1"/>
+<wire x1="12.7" y1="132.08" x2="5.08" y2="132.08" width="0.1524" layer="91"/>
+<label x="5.08" y="132.08" size="1.778" layer="95" rot="R180" xref="yes"/>
 </segment>
 </net>
@@
 <net name="HV" class="0">
 <segment>
-<pinref part="HVOUT" gate="G$1" pin="1"/>
-<wire x1="12.7" y1="132.08" x2="7.62" y2="132.08" width="0.1524" layer="91"/>
-<label x="7.62" y="132.08" size="1.778" layer="95" rot="R180" xref="yes"/>
-</segment>
-<segment>
 <pinref part="R4" gate="G$1" pin="2"/>
 <wire x1="86.36" y1="144.78" x2="86.36" y2="147.32" width="0.1524" layer="91"/>
 <label x="86.36" y="147.32" size="1.778" layer="95" rot="R90" xref="yes"/>
 </segment>
-</net>
-<net name="N$4" class="0">
-<segment>
-<pinref part="HVOUT" gate="G$1" pin="2"/>
-<wire x1="12.7" y1="129.54" x2="7.62" y2="129.54" width="0.1524" layer="91"/>
-</segment>
-</net>
-<net name="N$7" class="0">
-<segment>
-<pinref part="HVIN" gate="G$1" pin="2"/>
-<wire x1="12.7" y1="116.84" x2="7.62" y2="116.84" width="0.1524" layer="91"/>
+<segment>
+<pinref part="D3" gate="1" pin="C"/>
+<wire x1="0" y1="119.38" x2="-7.62" y2="119.38" width="0.1524" layer="91"/>
+<label x="-7.62" y="119.38" size="1.778" layer="95" rot="R180" xref="yes"/>
 </segment>
 </net>
@@
 </segment>
 </net>
+<net name="N$4" class="0">
+<segment>
+<pinref part="HVIN" gate="G$1" pin="1"/>
+<wire x1="12.7" y1="119.38" x2="5.08" y2="119.38" width="0.1524" layer="91"/>
+<pinref part="D3" gate="1" pin="A"/>
+</segment>
+</net>
